File: pcb/TGN.kicad_pcb (KiCad board)
At the start: 2 copper layers, 110.7 x 74.7 mm, 92 parts, among them J1 Screw_Terminal_01x02, J10 Conn_01x08_Pin, J11 Conn_01x03_Pin, J12 Conn_01x03_Pin, J2 Conn_01x02_Pin, J3 Conn_01x02_Pin, J4 Conn_01x02_Pin, J5 Screw_Terminal_01x02, J6 Conn_01x03_Pin, J7 Screw_Terminal_01x02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

Commit message: Adapt ladder resistor values
Parts:
- R13, R14, R15, R16, R17, R18, R19: value 10k -> 1k
- R20, R21, R22, R23, R24, R25, R26, R27, R28: value 20k -> 2k
Changed lines of the file:
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@@
     (property "Sheetname" "Memory")
     (property "Vendor" "DigiKey")
-    (property "VendorId" "13-MFR-25FRF52-20KCT-ND")
+    (property "VendorId" "13-MFR-25FRF52-2KCT-ND")
     (property "ki_description" "Resistor")
     (property "ki_keywords" "R res resistor")
@@
         (effects (font (size 1 1) (thickness 0.15)))
     )
-    (fp_text value "20k" (at -1.607721 0 90) (layer "F.Fab")
+    (fp_text value "2k" (at -1.607721 0 90) (layer "F.Fab")
         (effects (font (size 1 1) (thickness 0.15)))
     )
@@
     (property "Sheetname" "Memory")
     (property "Vendor" "DigiKey")
-    (property "VendorId" "13-MFR-25FRF52-20KCT-ND")
+    (property "VendorId" "13-MFR-25FRF52-2KCT-ND")
     (property "ki_description" "Resistor")
     (property "ki_keywords" "R res resistor")
@@
         (effects (font (size 1 1) (thickness 0.15)))
     )
-    (fp_text value "20k" (at -1.607721 0 90) (layer "F.Fab")
+    (fp_text value "2k" (at -1.607721 0 90) (layer "F.Fab")
         (effects (font (size 1 1) (thickness 0.15)))
     )
@@
     (property "Sheetname" "Memory")
     (property "Vendor" "DigiKey")
-    (property "VendorId" "13-MFR-25FRF52-20KCT-ND")
+    (property "VendorId" "13-MFR-25FRF52-2KCT-ND")
     (property "ki_description" "Resistor")
     (property "ki_keywords" "R res resistor")
@@
         (effects (font (size 1 1) (thickness 0.15)))
     )
-    (fp_text value "20k" (at 5.08 2.37 90) (layer "F.Fab")
+    (fp_text value "2k" (at 5.08 2.37 90) (layer "F.Fab")
         (effects (font (size 1 1) (thickness 0.15)))
     )
@@
     (property "Sheetname" "Memory")
     (property "Vendor" "HTL")
-    (property "VendorId" "102812")
+    (property "VendorId" "102800")
     (property "ki_description" "Resistor")
     (property "ki_keywords" "R res resistor")
@@
         (effects (font (size 1 1) (thickness 0.15)))
     )
-    (fp_text value "10k" (at 12.362279 0 90) (layer "F.Fab")
+    (fp_text value "1k" (at 12.362279 0 90) (layer "F.Fab")
         (effects (font (size 1 1) (thickness 0.15)))
     )
@@
     (property "Sheetname" "Memory")
     (property "Vendor" "HTL")
-    (property "VendorId" "102812")
+    (property "VendorId" "102800")
     (property "ki_description" "Resistor")
     (property "ki_keywords" "R res resistor")
@@
         (effects (font (size 1 1) (thickness 0.15)))
     )
-    (fp_text value "10k" (at 12.362279 0 90) (layer "F.Fab")
+    (fp_text value "1k" (at 12.362279 0 90) (layer "F.Fab")
         (effects (font (size 1 1) (thickness 0.15)))
     )
@@
     (property "Sheetname" "Memory")
     (property "Vendor" "DigiKey")
-    (property "VendorId" "13-MFR-25FRF52-20KCT-ND")
+    (property "VendorId" "13-MFR-25FRF52-2KCT-ND")
     (property "ki_description" "Resistor")
     (property "ki_keywords" "R res resistor")
@@
         (effects (font (size 1 1) (thickness 0.15)))
     )
-    (fp_text value "20k" (at -1.607721 0 90) (layer "F.Fab")
+    (fp_text value "2k" (at -1.607721 0 90) (layer "F.Fab")
         (effects (font (size 1 1) (thickness 0.15)))
     )
@@
     (property "Sheetname" "Memory")
     (property "Vendor" "DigiKey")
-    (property "VendorId" "13-MFR-25FRF52-20KCT-ND")
+    (property "VendorId" "13-MFR-25FRF52-2KCT-ND")
     (property "ki_description" "Resistor")
     (property "ki_keywords" "R res resistor")
@@
         (effects (font (size 1 1) (thickness 0.15)))
     )
-    (fp_text value "20k" (at -1.607721 0 90) (layer "F.Fab")
+    (fp_text value "2k" (at -1.607721 0 90) (layer "F.Fab")
         (effects (font (size 1 1) (thickness 0.15)))
     )
@@
     (property "Sheetname" "Memory")
     (property "Vendor" "HTL")
-    (property "VendorId" "102812")
+    (property "VendorId" "102800")
     (property "ki_description" "Resistor")
     (property "ki_keywords" "R res resistor")
@@
         (effects (font (size 1 1) (thickness 0.15)))
     )
-    (fp_text value "10k" (at 12.362279 0 90) (layer "F.Fab")
+    (fp_text value "1k" (at 12.362279 0 90) (layer "F.Fab")
         (effects (font (size 1 1) (thickness 0.15)))
     )
@@
     (property "Sheetname" "Memory")
     (property "Vendor" "HTL")
-    (property "VendorId" "102812")
+    (property "VendorId" "102800")
     (property "ki_description" "Resistor")
     (property "ki_keywords" "R res resistor")
@@
         (effects (font (size 1 1) (thickness 0.15)))
     )
-    (fp_text value "10k" (at 12.362279 0 90) (layer "F.Fab")
+    (fp_text value "1k" (at 12.362279 0 90) (layer "F.Fab")
         (effects (font (size 1 1) (thickness 0.15)))
     )
@@
     (property "Sheetname" "Memory")
     (property "Vendor" "HTL")
-    (property "VendorId" "102812")
+    (property "VendorId" "102800")
     (property "ki_description" "Resistor")
     (property "ki_keywords" "R res resistor")
@@
         (effects (font (size 1 1) (thickness 0.15)))
     )
-    (fp_text value "10k" (at 12.362279 0 90) (layer "F.Fab")
+    (fp_text value "1k" (at 12.362279 0 90) (layer "F.Fab")
         (effects (font (size 1 1) (thickness 0.15)))
     )
@@
     (property "Sheetname" "Memory")
     (property "Vendor" "DigiKey")
-    (property "VendorId" "13-MFR-25FRF52-20KCT-ND")
+    (property "VendorId" "13-MFR-25FRF52-2KCT-ND")
     (property "ki_description" "Resistor")
     (property "ki_keywords" "R res resistor")
@@
         (effects (font (size 1 1) (thickness 0.15)))
     )
-    (fp_text value "20k" (at -1.607721 0 90) (layer "F.Fab")
+    (fp_text value "2k" (at -1.607721 0 90) (layer "F.Fab")
         (effects (font (size 1 1) (thickness 0.15)))
     )
@@
     (property "Sheetname" "Memory")
     (property "Vendor" "DigiKey")
-    (property "VendorId" "13-MFR-25FRF52-20KCT-ND")
+    (property "VendorId" "13-MFR-25FRF52-2KCT-ND")
     (property "ki_description" "Resistor")
     (property "ki_keywords" "R res resistor")
@@
         (effects (font (size 1 1) (thickness 0.15)))
     )
-    (fp_text value "20k" (at -1.607721 0 90) (layer "F.Fab")
+    (fp_text value "2k" (at -1.607721 0 90) (layer "F.Fab")
         (effects (font (size 1 1) (thickness 0.15)))
     )
@@
     (property "Sheetname" "Memory")
     (property "Vendor" "HTL")
-    (property "VendorId" "102812")
+    (property "VendorId" "102800")
     (property "ki_description" "Resistor")
     (property "ki_keywords" "R res resistor")
@@
         (effects (font (size 1 1) (thickness 0.15)))
     )
-    (fp_text value "10k" (at 12.362279 0 90) (layer "F.Fab")
+    (fp_text value "1k" (at 12.362279 0 90) (layer "F.Fab")
         (effects (font (size 1 1) (thickness 0.15)))
     )
@@
     (property "Sheetname" "Memory")
     (property "Vendor" "HTL")
-    (property "VendorId" "102812")
+    (property "VendorId" "102800")
     (property "ki_description" "Resistor")
     (property "ki_keywords" "R res resistor")
@@
         (effects (font (size 1 1) (thickness 0.15)))
     )
-    (fp_text value "10k" (at 12.362279 0 90) (layer "F.Fab")
+    (fp_text value "1k" (at 12.362279 0 90) (layer "F.Fab")
         (effects (font (size 1 1) (thickness 0.15)))
     )
@@
     (property "Sheetname" "Memory")
     (property "Vendor" "DigiKey")
-    (property "VendorId" "13-MFR-25FRF52-20KCT-ND")
+    (property "VendorId" "13-MFR-25FRF52-2KCT-ND")
     (property "ki_description" "Resistor")
     (property "ki_keywords" "R res resistor")
@@
         (effects (font (size 1 1) (thickness 0.15)))
     )
-    (fp_text value "20k" (at 12.362279 0 90) (layer "F.Fab")
+    (fp_text value "2k" (at 12.362279 0 90) (layer "F.Fab")
         (effects (font (size 1 1) (thickness 0.15)))
     )
@@
     (property "Sheetname" "Memory")
     (property "Vendor" "DigiKey")
-    (property "VendorId" "13-MFR-25FRF52-20KCT-ND")
+    (property "VendorId" "13-MFR-25FRF52-2KCT-ND")
     (property "ki_description" "Resistor")
     (property "ki_keywords" "R res resistor")
@@
         (effects (font (size 1 1) (thickness 0.15)))
     )
-    (fp_text value "20k" (at -1.607721 0 90) (layer "F.Fab")
+    (fp_text value "2k" (at -1.607721 0 90) (layer "F.Fab")
         (effects (font (size 1 1) (thickness 0.15)))
     )
